File: ecad/LC_meter/analog_front_end.kicad_sch (KiCad schematic)
At the start: 62 parts, among them J1 DUT, Q1 2N7000, Q2 2N7000, SW1 SW_SP3T, U1 LMC6484, U2 LMC6482, U3 LM385BZ-2.5, U4 MCP3204, U6 LTC1044, U7 LMC6484

Commit message: schematic work
Parts:
- removed C11: 0.1uF, symbol Device:C
- removed C12, C13: 10uF, symbol Device:C
- removed D2 (x2), D4 (x2): BAS33, symbol Device:D
- removed Q1, Q2: 2N7000, Package_TO_SOT_THT:TO-92_Inline, symbol Transistor_FET:2N7000
- removed R12, R8: 10k, symbol Device:R_US
- removed R13, R9: 1k, symbol Device:R_US
- removed SW1: SW_SP3T, symbol Switch:SW_SP3T
- removed unit 1 of U2
- removed unit 3 of U2
- removed U6: LTC1044, symbol Regulator_SwitchedCapacitor:LTC1044
- removed U7: LMC6484, symbol Amplifier_Operational:LMC6484
- added D1, D2, D4, D5: SSTPAD5, symbol LC_meter_parts:SSTPAD5
- added D8: SMF6.0CA, Diode_SMD:D_SMB, symbol Device:D_TVS
- added J4: Resistor Range, symbol Connector:Screw_Terminal_01x06
- added J5: Sine Wave, TerminalBlock_Phoenix:TerminalBlock_Phoenix_MPT-0,5-2-2.54_1x02_P2.54mm_Horizontal, symbol Connector:Screw_Terminal_01x02
- added K1: Relay_DPDT, symbol Relay:Relay_DPDT
- added R5: 700k+/-0.1%, Resistor_SMD:R_0805_2012Metric, symbol Device:R_US
- added R5: 7M+/-0.1%, Resistor_SMD:R_0805_2012Metric, symbol Device:R_US
- added R5: 70k+/-0.1%, Resistor_SMD:R_0805_2012Metric, symbol Device:R_US
- added TP5, TP6, TP7: TestPoint, symbol Connector:TestPoint
- added unit 5 of U1
- added unit 2 of U1
- added unit 3 of U2
- added unit 1 of U2
- added unit 4 of U2
- C1, C11, C2, C3, C4, C5, C6, C7, C8, C9: footprint (none) -> Capacitor_SMD:C_0805_2012Metric
- C18: footprint (none) -> Diode_SMD:D_0805_2012Metric
- J1: footprint (none) -> TerminalBlock_Phoenix:TerminalBlock_Phoenix_MPT-0,5-2-2.54_1x02_P2.54mm_Horizontal
- R1, R2, R30, R31: value 10k +/- 0.1% -> 10k+/-0.1%; footprint (none) -> Resistor_SMD:R_0805_2012Metric
- R1, R10, R11, R16, R2, R21, R22, R23, R24, R25, R26, R27, R3, R32, R33, R4, R6, R7: footprint (none) -> Resistor_SMD:R_0805_2012Metric
- R5: value 10k -> 700+/0.1%; footprint (none) -> Resistor_SMD:R_0805_2012Metric
- R5: value 10M -> 7k+/-0.1%; footprint (none) -> Resistor_SMD:R_0805_2012Metric
- R5: value 100 -> 70+/-0.1%; footprint (none) -> Resistor_SMD:R_0805_2012Metric
- TP1: footprint (none) -> Diode_SMD:D_SMB
Connections:
- net +5V: now also U1.4 (V+)
- net -5V: now also U1.11 (V-)
- net GND: now also D8.1 (A1), K1.11, K1.21, U2.3 (+)
- net at C18.2, R1.1, R2.2: now also U2.9 (-); no longer U2.6 (-)
- net at C18.1, R1.2, U1.10 (+): now also TP6.1, U2.8; no longer U2.7
- net at C4.1, R6.2, R7.1: now also U1.5 (+); no longer U1.12 (+)
- net at R21.1, R6.2, TP1.1: now also U1.6 (-), U1.7; no longer U1.13 (-), U1.14
- net at R30.1, R31.2: now also U2.10 (+); no longer U2.5 (+)
- net at J1.2 (Pin_2), R5.2, R5.2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: now also U2.5 (+), D8.2 (A2), R5.2, R5.2, R5.2, TP7.1
- net at R2.1: now also U2.6 (-), U2.7
- net at C3.1, R1.2, R25.1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: now also J5.1 (Pin_1), J5.2 (Pin_2), TP5.1, U2.1
- net at R6.1, U1.2 (-): now also D4.3
- net at R10.2, R23.1, TP2.1: now also U1.13 (-), U1.14
- net at U1.8: now also D1.1, D1.2, D2.3
- net at R10.1, U1.9 (-): now also D1.3
- net at C5.1, R10.2, R11.1: now also U1.12 (+)
- net at R32.2, R33.2: now also U2.12 (+)
- net at R1.1, R2.2: now also U2.2 (-)
- net at R5.1: now also J4.3 (Pin_3)
- net at R5.1: now also J4.2 (Pin_2)
- net at R5.1: now also J4.1 (Pin_1)
- net at R10.1: now also D2.1, D2.2
- net at R7.2: now also K1.14
- net at U1.1: now also D4.1, D4.2, D5.3
- net at R6.1: now also D5.1, D5.2
- net at R11.2: now also K1.24
- new net: J4.5 (Pin_5), R5.1
- new net: J4.4 (Pin_4), R5.1
- new net: J4.6 (Pin_6), R5.1
- new net: U2.13 (-), U2.14
Other:
- moved on the sheet: C11, C18, C4, C5, C6, C7, J1, R1, R10, R11, R16, R2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

Commit message: switch to time based
Parts:
- removed C18: 0.01uF, Diode_SMD:D_0805_2012Metric, symbol Device:C
- removed R1, R2, R30, R31: 10k+/-0.1%, Resistor_SMD:R_0805_2012Metric, symbol Device:R_US
- removed unit 3 of U2
- removed unit 2 of U2
- added D9: B220, Diode_SMD:D_SMB, symbol Diode:B220
- added Q1: 2N7002, Package_TO_SOT_SMD:SOT-23, symbol Transistor_FET:2N7002
- added R12: 1k, symbol Device:R_US
- added R13: 10k, symbol Device:R_US
- C1, C2, C3: value 0.1uF -> 1nF
- K1: value Relay_DPDT -> SR5-5V-200-1C
Connections:
- net +5V: now also K1.A1, D9.1 (K)
- net GND: now also Q1.2 (S), R13.2
- net at D8.2 (A2), J1.2 (Pin_2), R5.2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: now also TP6.1, U1.10 (+)
- net at K1.A2: now also D9.2 (A), Q1.3 (D)
- new net: Q1.1 (G), R12.2
- new net reset: R12.1, R13.1
Other:
- note removed: "Got to get that high Z!"
- moved on the sheet: C4, D4, D5, D8, J1, J4, J5, K1, R21, R22, R27, R32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
