File: ecad/LC_meter/time_analog_front_end.kicad_sch (KiCad schematic)
At the start: 33 parts, among them J10 Step Function, J11 Screw_Terminal_01x04, J6 Screw_Terminal_01x04, J7 Step Function, J8 DUT, J9 GND, SW1 SW_SPDT, SW2 SW_SPDT, U10 LMV7271, U7 LMV7271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

Commit message: time stuff
Parts:
- removed C18, C19, C20, C21: 0.1uF, symbol Device:C
- removed J10, J7: Step Function, symbol Connector:Screw_Terminal_01x02
- removed J11, J6: Screw_Terminal_01x04, symbol Connector:Screw_Terminal_01x04
- removed J8: DUT, symbol Connector:Screw_Terminal_01x02
- removed J9: GND, symbol Connector:Screw_Terminal_01x02
- removed R1, R55, R58: 100k, symbol Device:R_US
- removed R14, R15, R2, R47, R54, R57: 10k, symbol Device:R_US
- removed R5 (x2): 10M, Resistor_SMD:R_0805_2012Metric, symbol Device:R_US
- removed R5 (x2): 100k, Resistor_SMD:R_0805_2012Metric, symbol Device:R_US
- removed R5 (x4): TBD, Resistor_SMD:R_0805_2012Metric, symbol Device:R_US
- removed SW1, SW2: SW_SPDT, symbol Switch:SW_SPDT
- removed U10, U7: LMV7271, symbol Comparator:LMV7271
- removed U8, U9: Opamp_Dual, symbol Device:Opamp_Dual
