File: ecad/LC_meter/acquisition.kicad_sch (KiCad schematic)
At the start: 54 parts, among them J1 DUT, Q1 2N7000, Q2 2N7000, SW1 SW_SP3T, SW2 SW_SP3T, U1 LM6144xIx, U2 LM6144xIx, U7 LM6144xIx, U8 LM6144xIx, U9 MCP3422

Commit message: ok range calcs and schematic
Parts:
- removed C1, C11, C2, C3, C4, C5, C6, C7, C8, C9: 0.1uF, symbol Device:C
- removed D2 (x2), D4 (x2): BAS33, symbol Device:D
- removed J1: DUT, symbol Connector:Screw_Terminal_01x02
- removed Q1, Q2: 2N7000, Package_TO_SOT_THT:TO-92_Inline, symbol Transistor_FET:2N7000
- removed R1: 187k, symbol Device:R_US
- removed R10 (x2), R13, R6 (x2), R9: 1k, symbol Device:R_US
- removed R11, R5 (x2), R7: 100, symbol Device:R_US
- removed R12, R26, R30, R31, R32, R5 (x2), R8: 10k, symbol Device:R_US
- removed R2, R3, R4: 6.49k, symbol Device:R_US
- removed R21, R23: 1.5k+/-0.1%, symbol Device:R_US
- removed R22, R24: 1k+/-0.1%, symbol Device:R_US
- removed R5 (x2): 10M, symbol Device:R_US
- removed SW1, SW2: SW_SP3T, symbol Switch:SW_SP3T
- removed TP1, TP2: TestPoint, symbol Connector:TestPoint
- removed U1, U2, U7, U8: LM6144xIx, symbol Amplifier_Operational:LM6144xIx
- removed U9: MCP3422, symbol Analog_ADC:MCP3422
