File: ecad/LC_meter.kicad_pcb (KiCad board)
At the start: 2 copper layers, 77.7 x 77 mm, 75 parts, among them J1 DUT, J10 Range Switch, J11 Range Switch, J12 Display Connector, J2 Switch, J3 12V Power, J4 Switch, J6 Switch, J7 Switch, J8 Thevenin Range Switch Indicat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

Commit message: fished crash
Parts:
- moved C4 5.43 mm to (162.0, 123.4)
- moved R9 5.43 mm to (169.8, 119.9)
- moved C2 5.43 mm to (165.0, 119.0)
- moved C3 5.43 mm to (162.9, 120.6)
- moved C5 5.43 mm to (168.4, 114.8)
- moved R10 5.43 mm to (160.0, 121.3)
- moved R12 5.43 mm to (162.1, 114.2)
- moved R4 5.43 mm to (162.9, 117.0)
- moved R8 5.43 mm to (158.2, 119.3)
- moved R11 3.66 mm to (165.6, 123.4)
- moved TP6 3.26 mm to (175.1, 115.2)
- moved U1 3.26 mm to (158.8, 111.0)
- moved C11 0.46 mm to (143.8, 92.3)
- moved R23 0.10 mm to (139.4, 115.0)
Routing:
- net Net-(J9-Pin_2): track 0.00 -> 42.3 mm, vias 0 -> 4
- net Net-(J9-Pin_3): track 0.00 -> 35.6 mm, vias 0 -> 4
- net Net-(J9-Pin_4): track 0.00 -> 33.0 mm, vias 0 -> 2
- net GNDA: track 15.1 -> 20.6 mm
- net Net-(U1B--): track 2.54 -> 7.20 mm
- net Net-(U2-K): track 0.00 -> 4.07 mm
- net Net-(U1A--): track 4.50 -> 1.93 mm
- net Net-(J11-Pin_1): track 4.78 -> 7.32 mm
- net GNDD: track 22.1 -> 24.1 mm, vias 11 -> 12
- net Net-(C3-Pad1): track 5.47 -> 3.77 mm
- net Net-(J2-Pin_1): track 16.1 -> 14.4 mm

Commit message: layout
Parts:
- U4: footprint Package_SO:TSSOP-14-1EP_4.4x5mm_P0.65mm -> Package_SO:TSSOP-16_4.4x5mm_P0.65mm
- moved TP7 22.8 mm to (154.0, 81.7)
- moved R17 12.7 mm to (142.3, 87.2)
- moved U2 10.7 mm to (154.0, 86.9), turned to -90 degrees
- moved C9 9.89 mm to (153.9, 90.2), turned to 0 degrees
- moved R18 9.80 mm to (153.1, 93.0), turned to 90 degrees
- moved C8 9.54 mm to (148.0, 96.7), turned to -90 degrees
- moved J1 8.54 mm to (163.0, 129.0)
- moved J6 7.64 mm to (160.3, 87.0), turned to -90 degrees
- moved TP2 6.11 mm to (142.1, 80.8)
- moved TP5 6.07 mm to (147.9, 85.4)
- moved R23 5.49 mm to (144.0, 118.0), turned to 0 degrees
- moved C17 5.48 mm to (151.0, 117.3)
- moved C16 5.47 mm to (148.7, 117.3)
- moved U8 5.47 mm to (151.0, 125.5)
- moved TP1 5.11 mm to (149.7, 108.0)
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Connections:
- C11 pad 2: GNDA -> GNDD
- J12 pad 1: +5V -> +3.3V
Routing:
- net Net-(J1-Pin_2): track 7.61 -> 74.8 mm, vias 0 -> 1
- net Net-(J2-Pin_1): track 14.4 -> 64.4 mm
- net /Analog Front End/SCK: track 0.00 -> 45.7 mm, vias 0 -> 2
- net Net-(D5-K): track 9.87 -> 54.6 mm
- net Net-(U4-+IN1): track 22.8 -> 65.1 mm, vias 0 -> 4
- net Net-(J1-Pin_1): track 25.6 -> 63.0 mm, vias 0 -> 2
- net Net-(U1B--): track 7.20 -> 43.9 mm, vias 0 -> 2
- net /Analog Front End/INTERUPT: track 0.00 -> 32.5 mm, vias 0 -> 4
- net /SDA: track 5.09 -> 36.5 mm, vias 0 -> 2
- net /Analog Front End/DATA_IN: track 0.00 -> 31.4 mm, vias 0 -> 4
- net /Analog Front End/CS: track 2.14 -> 32.8 mm, vias 0 -> 4
- net /Analog Front End/DATA_OUT: track 0.00 -> 29.7 mm, vias 0 -> 4
- net /SCL: track 4.95 -> 32.6 mm, vias 0 -> 2
- net /Analog Front End/V/2: track 18.1 -> 43.0 mm, vias 0 -> 2
- net Net-(U2-K): track 4.07 -> 18.9 mm
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Other:
- board size 77.7 x 77 mm -> 78 x 77 mm

Commit message: more layout
Parts:
- moved R8 10.5 mm to (167.5, 121.7), turned to 0 degrees
- moved C4 6.14 mm to (158.3, 116.0)
- moved R23 4.00 mm to (144.1, 114.0)
- moved R12 3.96 mm to (163.9, 113.4)
- moved R9 2.34 mm to (167.5, 119.6)
- moved R15 2.06 mm to (160.2, 100.4), turned to -90 degrees
- moved C3 1.87 mm to (163.9, 119.6), turned to 0 degrees
- moved R11 1.82 mm to (164.0, 121.7)
- moved C2 1.44 mm to (163.9, 117.5), turned to 180 degrees
- moved R4 1.39 mm to (163.9, 115.4), turned to 0 degrees
- moved R10 0.81 mm to (158.3, 119.6)
- moved R16 0.72 mm to (162.3, 100.4), turned to 90 degrees
- moved C5 0.34 mm to (166.8, 114.1)
Routing:
- net +5V: track 5.98 -> 23.7 mm, vias 2 -> 8
- net Net-(J2-Pin_1): track 64.4 -> 57.1 mm
- net Net-(C2-Pad1): track 12.0 -> 6.00 mm
- net GNDA: track 30.4 -> 33.2 mm
- net Net-(U1A--): track 4.94 -> 7.10 mm
- net Net-(C3-Pad1): track 7.63 -> 9.52 mm
- net +3.3V: track 0.00 -> 1.69 mm
- net Net-(U1D-+): track 6.94 -> 5.27 mm
- net Net-(D2-K): track 10.6 -> 9.49 mm
- net Net-(J1-Pin_2): track 74.8 -> 75.4 mm

Commit message: general work
Parts:
- added J13: Mode Switch, TerminalBlock_Phoenix:TerminalBlock_Phoenix_MPT-0,5-2-2.54_1x02_P2.54mm_Horizontal, F.Cu at (116.5, 53.0)
- added J14: Panel LED, TerminalBlock_Phoenix:TerminalBlock_Phoenix_MPT-0,5-2-2.54_1x02_P2.54mm_Horizontal, F.Cu at (139.0, 128.0)
- added J5: Mode Switch, TerminalBlock_Phoenix:TerminalBlock_Phoenix_MPT-0,5-2-2.54_1x02_P2.54mm_Horizontal, F.Cu at (106.0, 59.5)
- added Q1: 2N7002, Package_TO_SOT_SMD:SOT-23, F.Cu at (136.2, 121.8)
- added R21: 68, Resistor_SMD:R_0805_2012Metric, F.Cu at (142.0, 121.9)
- added R22: 10k, Resistor_SMD:R_0805_2012Metric, F.Cu at (137.2, 117.8)
- added R24: 10k, Resistor_SMD:R_0805_2012Metric, F.Cu at (112.0, 63.0)
- added R25: 10k, Resistor_SMD:R_0805_2012Metric, F.Cu at (112.0, 59.0)
- C13, C14, R19, R20: value TBD -> PNU
- C6, C7: value C -> PNU
- R13: value 1e3+/-0.1% -> 250+/-0.1%
- R14: value 330+/-0.1% -> 2.5k+/-0.1%
- moved H1 7.00 mm to (175.0, 53.0)
- moved H2 7.00 mm to (105.0, 53.0)
Connections:
- J10 pad 1: Net-(J10-Pin_1) -> +3.3V
- J10 pad 2: Net-(J10-Pin_1) -> +3.3V
- J11 pad 1: Net-(J11-Pin_1) -> +3.3V
- J11 pad 2: Net-(J11-Pin_1) -> +3.3V
- U3 pad 1: unconnected-(U3-GP0-Pad1) -> Net-(J5-Pin_2)
- U3 pad 2: unconnected-(U3-GP1-Pad2) -> Net-(J13-Pin_2)
- U3 pad 22: unconnected-(U3-GP17-Pad22) -> Net-(U3-GP17)
Routing:
- net Net-(J13-Pin_2): track 0.00 -> 19.0 mm
- net Net-(J5-Pin_2): track 0.00 -> 15.0 mm
- net Net-(U3-GP17): track 0.00 -> 14.8 mm, vias 0 -> 2
- net Net-(J14-Pin_2): track 0.00 -> 8.53 mm
- net Net-(J14-Pin_1): track 0.00 -> 7.89 mm
- net Net-(J10-Pin_1): track 7.13 -> 4.59 mm
- net Net-(Q1-G): track 0.00 -> 2.13 mm
- net GNDD: track 37.4 -> 39.1 mm, vias 17 -> 18
Other:
- board size 78 x 77 mm -> 78 x 84 mm

Commit message: layout draft
Parts:
- removed the R21 at (111.8, 99.1)
- removed the R22 at (111.8, 82.1)
- added C15: 0.1uF, Capacitor_SMD:C_0805_2012Metric, F.Cu at (173.3, 88.4)
- added R26: 2.21k, Resistor_SMD:R_0805_2012Metric, F.Cu at (173.4, 96.8)
- added R27: 10k, Resistor_SMD:R_0805_2012Metric, F.Cu at (173.4, 94.7)
- added R30: 10k, Resistor_SMD:R_0805_2012Metric, F.Cu at (173.4, 90.5)
- added R31: 10k, Resistor_SMD:R_0805_2012Metric, F.Cu at (173.4, 92.6)
- added U6: LM6142xIx, Package_DIP:DIP-8_W7.62mm, F.Cu at (162.2, 94.8)
- R15: value 10k -> 2.21k
- R22: value 10k -> 1k
- moved TP5 32.3 mm to (176.4, 100.5)
- moved R15 19.4 mm to (173.4, 86.2), turned to 0 degrees
- moved C14 13.6 mm to (173.4, 84.1)
- moved C13 13.5 mm to (173.4, 80.0)
- moved C7 13.5 mm to (173.5, 75.8)
- moved J4 13.5 mm to (168.0, 67.1)
- moved J6 13.5 mm to (160.1, 73.5)
- moved J7 13.5 mm to (168.0, 81.1)
- moved R13 13.5 mm to (173.5, 69.6)
- moved R19 13.5 mm to (173.4, 77.9)
- moved R3 13.5 mm to (173.5, 67.2)
- moved R5 13.5 mm to (173.5, 64.7)
- moved J2 13.5 mm to (160.1, 59.5)
- moved C6 13.5 mm to (173.5, 71.7)
- moved R14 13.5 mm to (173.5, 73.7)
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Connections:
- C13 pad 2: Net-(U4-+IN1) -> Net-(C13-Pad2)
- C14 pad 2: Net-(U4-+IN1) -> Net-(C13-Pad2)
- C6 pad 2: Net-(U4-+IN1) -> Net-(C13-Pad2)
- C7 pad 2: Net-(U4-+IN1) -> Net-(C13-Pad2)
- R13 pad 2: Net-(U4-+IN1) -> Net-(C13-Pad2)
- R14 pad 2: Net-(U4-+IN1) -> Net-(C13-Pad2)
- R15 pad 1: +5V -> Net-(U1D-+)
- R15 pad 2: Net-(U1D-+) -> Net-(C13-Pad2)
- R19 pad 2: Net-(U4-+IN1) -> Net-(C13-Pad2)
- R20 pad 2: Net-(U4-+IN1) -> Net-(C13-Pad2)
- TP5 pad 1: Net-(U4-+IN1) -> Net-(C13-Pad2)
- U1 pad 8: Net-(U4-+IN1) -> Net-(C13-Pad2)
- U4 pad 2: Net-(U4-+IN1) -> Net-(U1D--)
- U4 pad 3: Net-(U1B--) -> Net-(U4-+IN0)
Routing:
- net Net-(U4-+IN1): track 65.1 -> 0.00 mm, vias 4 -> 0
- net Net-(C13-Pad2): track 0.00 -> 38.7 mm
- net Net-(U1D-+): track 5.27 -> 36.0 mm, vias 0 -> 2
- net Net-(U1B--): track 43.9 -> 23.5 mm, vias 2 -> 0
- net Net-(U1D--): track 2.54 -> 21.6 mm
- net Net-(J2-Pin_1): track 57.1 -> 76.0 mm, vias 0 -> 2
- net Net-(J1-Pin_2): track 75.4 -> 93.4 mm
- net Net-(U4-+IN0): track 0.00 -> 17.5 mm
- net Net-(J1-Pin_1): track 63.3 -> 80.1 mm, vias 2 -> 4
- net Net-(U6A-+): track 0.00 -> 9.10 mm
- net +5V: track 23.7 -> 32.4 mm, vias 8 -> 10
- net Net-(U6B-+): track 0.00 -> 7.90 mm
- net Net-(J11-Pin_1): track 7.32 -> 0.00 mm
- net Net-(J10-Pin_1): track 4.59 -> 0.00 mm
- net /Analog Front End/V/2: track 43.0 -> 47.5 mm, vias 2 -> 0
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
Commit message: finished algorithm
Parts:
- added TP10: 4952, Connector_Pin:Pin_D1.2mm_L10.2mm_W2.9mm_FlatFork, F.Cu at (190.8, 77.4)
- added TP11: 4952, Connector_Pin:Pin_D1.2mm_L10.2mm_W2.9mm_FlatFork, F.Cu at (187.3, 94.6)
- added TP12: 4952, Connector_Pin:Pin_D1.2mm_L10.2mm_W2.9mm_FlatFork, F.Cu at (158.6, 79.7)
- added TP13: 4952, Connector_Pin:Pin_D1.2mm_L10.2mm_W2.9mm_FlatFork, F.Cu at (158.6, 96.4)
- added TP8: 4952, Connector_Pin:Pin_D1.2mm_L10.2mm_W2.9mm_FlatFork, F.Cu at (191.0, 99.9)
- added TP9: 4952, Connector_Pin:Pin_D1.2mm_L10.2mm_W2.9mm_FlatFork, F.Cu at (186.9, 81.2)
- R1, R16, R2, R27: value 10k -> 10k+/-0.1%
- R13: value 250+/-0.1% -> 249+/-0.1%
- R14: value 2.5k+/-0.1% -> 2.49k+/-0.1%
- R15, R26: value 2.21k -> 2.21k+/-0.1%
- R3: value 500+/-0.1% -> 499+/-0.1%
- R5: value 5k+/-0.1% -> 4.99k+/-0.1%
- R6: value 50k+/-0.1% -> 49.9k+/-0.1%
- R7: value 500k+/-0.1% -> 499k+/-0.1%
- moved TP2 53.3 mm to (187.0, 52.0)
- moved R23 49.8 mm to (193.8, 110.2)
- moved R17 48.8 mm to (191.0, 84.4)
- moved U4 48.8 mm to (193.9, 89.2)
- moved C11 48.8 mm to (190.7, 94.0)
- moved C8 48.8 mm to (196.7, 93.9)
- moved C16 48.2 mm to (196.9, 116.0)
- moved C17 48.2 mm to (199.2, 116.0)
- moved U8 48.2 mm to (199.2, 124.2)
- moved C10 46.3 mm to (176.0, 114.5)
- moved C13 46.3 mm to (219.7, 77.2)
- moved C15 46.3 mm to (219.6, 85.6)
- moved C2 46.3 mm to (210.2, 114.7)
- moved C3 46.3 mm to (210.2, 116.8)
- moved D5 46.3 mm to (167.0, 114.3)
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Connections:
- U3 pad 14: unconnected-(U3-GP10-Pad14) -> /Analog Front End/CONVST
- U4 pad 9: unconnected-(U4-CONVST-Pad9) -> /Analog Front End/CONVST
Routing:
- net /Analog Front End/CONVST: track 0.00 -> 45.6 mm, vias 0 -> 2
- net /Analog Front End/DATA_IN: track 31.4 -> 47.7 mm
- net /Analog Front End/SCK: track 46.0 -> 58.3 mm
- net /Analog Front End/CS: track 32.8 -> 43.6 mm
- net /Analog Front End/DATA_OUT: track 29.7 -> 40.3 mm
- net +5V: track 32.4 -> 41.5 mm, vias 10 -> 14
- net /Analog Front End/INTERUPT: track 32.4 -> 41.0 mm
- net /SCL: track 32.6 -> 26.0 mm
- net Net-(J2-Pin_1): track 76.0 -> 70.7 mm
- net Net-(U2-K): track 15.1 -> 20.1 mm
- net Net-(U1D--): track 21.6 -> 17.2 mm
- net Net-(U4-+IN0): track 17.5 -> 15.0 mm
- net /Analog Front End/V/2: track 47.5 -> 45.2 mm
- net Net-(D5-K): track 55.4 -> 56.9 mm
- net /SDA: track 36.5 -> 38.0 mm
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
Commit message: boms
Parts:
- moved H3 4.11 mm to (220.0, 130.0)
- moved H1 3.98 mm to (220.0, 54.0)
- moved H2 3.98 mm to (150.0, 54.0)
- moved H4 3.89 mm to (150.0, 130.0)
- moved C10 3.73 mm to (175.0, 118.1)
- moved C12 3.73 mm to (172.7, 118.1)
- moved C13 3.73 mm to (218.7, 80.8)
- moved C14 3.73 mm to (218.6, 84.9)
- moved C15 3.73 mm to (218.6, 89.2)
- moved C16 3.73 mm to (195.9, 119.6)
- moved C17 3.73 mm to (198.2, 119.6)
- moved C3 3.73 mm to (209.2, 120.4)
- moved C5 3.73 mm to (212.0, 114.9)
- moved C9 3.73 mm to (195.8, 85.7)
- moved D7 3.73 mm to (160.0, 125.3)
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Routing:
- net /SCL: track 26.0 -> 33.8 mm
