File: ecad/LC_meter.kicad_sch (KiCad schematic)
At the start: 31 parts, among them J10 Range Switch, J11 Range Switch, J12 Display Connector, J3 12V Power, J8 Thevenin Range Switch Indicat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, J9 Current Range Switch Indicator, U3 Raspberry Pi Pico SC0915, U5 LM1117DT-3.3, U8 LM1117DT-5.0

Commit message: layout
Connections:
- net +3.3V: now also J12.1 (Pin_1)
- net +5V: no longer J12.1 (Pin_1)
Changed lines of the file:
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@@
-    )
-  )
-  (symbol (lib_id "power:+5V") (at 184.15 118.11 0) (unit 1)
-    (in_bom yes) (on_board yes) (dnp no) (fields_autoplaced)
-    (property "Reference" "#PWR034" (at 184.15 121.92 0)
-      (effects (font (size 1.27 1.27)) hide)
-    )
-    (property "Value" "+5V" (at 184.15 113.03 0)
-      (effects (font (size 1.27 1.27)))
-    )
-    (property "Footprint" "" (at 184.15 118.11 0)
-      (effects (font (size 1.27 1.27)) hide)
-    )
-    (property "Datasheet" "" (at 184.15 118.11 0)
-      (effects (font (size 1.27 1.27)) hide)
-    )
-    (pin "1")
-    (instances
-      (project "LC_meter"
-        (path "/0c53b8cf-b94b-444b-8930-5f445eddf0f0"
-          (reference "#PWR034") (unit 1)
-        )
-      )
     )
   )
@@
         )
       )
+    )
+  )
+  (symbol (lib_id "power:+3.3V") (at 184.15 118.11 0) (unit 1)
+    (in_bom yes) (on_board yes) (dnp no) (fields_autoplaced)
+    (property "Reference" "#PWR034" (at 184.15 121.92 0)
+      (effects (font (size 1.27 1.27)) hide)
+    )
+    (property "Value" "+3.3V" (at 184.15 113.03 0)
+      (effects (font (size 1.27 1.27)))
+    )
+    (property "Footprint" "" (at 184.15 118.11 0)
+      (effects (font (size 1.27 1.27)) hide)
+    )
+    (property "Datasheet" "" (at 184.15 118.11 0)
+      (effects (font (size 1.27 1.27)) hide)
+    )
+    (pin "1")
+    (instances
+      (project "LC_meter"
+        (path "/0c53b8cf-b94b-444b-8930-5f445eddf0f0"
+          (reference "#PWR034") (unit 1)
+        )
+      )

Commit message: general work
Parts:
- added J13, J5: Mode Switch, TerminalBlock_Phoenix:TerminalBlock_Phoenix_MPT-0,5-2-2.54_1x02_P2.54mm_Horizontal, symbol Connector:Screw_Terminal_01x02
- added J14: Panel LED, TerminalBlock_Phoenix:TerminalBlock_Phoenix_MPT-0,5-2-2.54_1x02_P2.54mm_Horizontal, symbol Connector:Screw_Terminal_01x02
- added Q1: 2N7002, Package_TO_SOT_SMD:SOT-23, symbol Transistor_FET:2N7002
- added R24, R25: 10k, Resistor_SMD:R_0805_2012Metric, symbol Device:R_US
- R21: value 10k -> 68
Connections:
- net +3.3V: now also J10.1 (Pin_1), J10.2 (Pin_2), J11.1 (Pin_1), J11.2 (Pin_2), R24.1, R25.1; no longer R22.1
- net GNDD: now also J13.1 (Pin_1), J5.1 (Pin_1), Q1.2 (S)
- net at U3.1 (GP0): now also J5.2 (Pin_2), R24.2
- net at U3.2 (GP1): now also J13.2 (Pin_2), R25.2
- net at U3.22 (GP17): now also R22.1
- new net: J14.1 (Pin_1), R21.2
- new net: J14.2 (Pin_2), Q1.3 (D)
- new net: Q1.1 (G), R22.2
- no-connect marks 27 -> 24
Other:
- moved on the sheet: J10, J11, J12, R28, R29

Commit message: layout draft
Parts:
- R22: value 10k -> 1k
Changed lines of the file:
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@@
       (effects (font (size 1.27 1.27)))
     )
-    (property "Value" "10k" (at 213.36 59.69 90)
+    (property "Value" "1k" (at 213.36 59.69 90)
       (effects (font (size 1.27 1.27)))
     )

Commit message: more work on algorithm
Parts:
- C10, C12, C17: Distributor (none) -> DIGIKEY; Distributor Part # (none) -> 1276-1096-1-ND; Part # (none) -> CL21A106KOQNNNE; Unit Price (none) -> 0.1
- C16: Distributor (none) -> DIGIKEY; Distributor Part # (none) -> 1276-1003-1-ND; Part # (none) -> CL21B104KBCNNNC; Unit Price (none) -> 0.1
- H1, H2, H3, H4: Distributor (none) -> N/A; Distributor Part # (none) -> N/A; Part # (none) -> N/A; Price (none) -> N/A; Unit Price (none) -> N/A
- R21: Distributor (none) -> DIGIKEY; Distributor Part # (none) -> P68DACT-ND; Part # (none) -> ERA-6AEB680V; Unit Price (none) -> 0.32
- R22: Distributor (none) -> DIGIKEY; Distributor Part # (none) -> RMCF0805FT1K00CT-ND; Part # (none) -> RMCF0805FT1K00; Unit Price (none) -> 0.1
- R23: Distributor (none) -> DIGIKEY; Distributor Part # (none) -> RMCF0805ZT0R00CT-ND; Part # (none) -> RMCF0805ZT0R00; Unit Price (none) -> 0.1
- R24, R25, R28, R29: Distributor (none) -> DIGIKEY; Distributor Part # (none) -> RMCF0805FT10K0CT-ND; Part # (none) -> RMCF0805FT10K0; Unit Price (none) -> 0.1
- R38: Distributor (none) -> DIGIKEY; Distributor Part # (none) -> YAG4850CT-ND; Part # (none) -> RT0805BRD071K78L; Unit Price (none) -> 0.36
- TP1, TP2, TP3: Distributor (none) -> DIGIKEY; Distributor Part # (none) -> 36-4952-ND; Part # (none) -> 4952; Unit Price (none) -> 0.26
- U3: Availability In Stock -> (none); Check_prices https://www.snapeda.com/parts/SC0915/Raspberry+Pi/view-part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 -> (none); MANUFACTURER Pi Supply -> (none); MF Raspberry Pi -> (none); MP SC0915 -> (none); PARTREV 1.9 -> (none); Package None -> (none); Price None -> (none); Purchase-URL https://www.snapeda.com/api/url_track_click_mouser/?unipart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 -> (none); SNAPEDA_PN SC0915 -> (none); STANDARD Manufacturer Recommendations -> (none); SnapEDA_Link https://www.snapeda.com/parts/SC0915/Raspberry+Pi/view-part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 -> (none)

Commit message: finished algorithm
Parts:
- added TP10, TP11, TP12, TP13, TP8, TP9: 4952, Connector_Pin:Pin_D1.2mm_L10.2mm_W2.9mm_FlatFork, symbol Connector:TestPoint_Alt
Connections:
- net Analog Front End/CS: now also TP12.1
- net Analog Front End/DATA_IN: now also TP10.1
- net Analog Front End/DATA_OUT: now also TP11.1
- net Analog Front End/INTERUPT: now also TP9.1
- net Analog Front End/SCK: now also TP8.1
- net Analog Front End/CONVST: now reaches U3.14 (GP10)
- net Analog Front End/CONVST: now also TP13.1
- no-connect marks 24 -> 23
Other:
- sheet Analog Front End ports: added CONVST; removed none

Commit message: boms
Parts:
- D1, D5: Distributor (none) -> DIGIKEY; Distributor Part # (none) -> B140-FDICT-ND; Part # (none) -> B140-13-F; Unit Price (none) -> 0.39
- D2: Distributor (none) -> DIGIKEY; Distributor Part # (none) -> SMF13A-TPMSCT-ND; Part # (none) -> SMF13A-TP; Unit Price (none) -> 0.38
- D7: Distributor (none) -> DIGIKEY; Distributor Part # (none) -> 160-1645-1-ND; Part # (none) -> LTST-C171TBKT; Unit Price (none) -> 0.32
- F1: Distributor (none) -> DIGIKEY; Distributor Part # (none) -> 507-1894-1-ND; Part # (none) -> 0685T2000-01; Unit Price (none) -> 0.32
- J10, J11, J13, J14, J3, J5: Distributor (none) -> DIGIKEY; Distributor Part # (none) -> ED10561-ND; Part # (none) -> OSTVN02A150; Unit Price (none) -> 1.08
- J12, J8, J9: Distributor (none) -> DIGIKEY; Distributor Part # (none) -> ED10563-ND; Part # (none) -> OSTVN04A150; Unit Price (none) -> 1.64
- Q1: Distributor (none) -> DIGIKEY; Distributor Part # (none) -> 2N7002NCT-ND; Part # (none) -> 2N7002; Unit Price (none) -> 0.45
- U3: Distributor (none) -> DIGIKEY; Distributor Part # (none) -> 2648-SC0915CT-ND; Part # (none) -> SC0915; Unit Price (none) -> 4
- U5: Distributor (none) -> DIGIKEY; Distributor Part # (none) -> LM1117DT-3.3/NOPB-ND; Part # (none) -> LM1117DT-3.3/NOPB; Unit Price (none) -> 1.81
- U8: Distributor (none) -> DIGIKEY; Distributor Part # (none) -> LM1117DT-5.0/NOPB-ND; Part # (none) -> LM1117DT-5.0/NOPB; Unit Price (none) -> 1.81
