File: ecad/analog_front_end.kicad_sch (KiCad schematic)
At the start: 44 parts, among them J1 DUT, J2 Switch, J4 Switch, J6 Switch, J7 Switch, U1 LM6144xIx, U2 LM4030-4.096, U4 ADS8328IPW

Commit message: layout
Parts:
- U4: footprint Package_SO:TSSOP-14-1EP_4.4x5mm_P0.65mm -> Package_SO:TSSOP-16_4.4x5mm_P0.65mm
Connections:
- net GNDA: no longer C11.2
- net GNDD: now also C11.2
Changed lines of the file:
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@@
       (effects (font (size 1.27 1.27)))
     )
-    (property "Footprint" "Package_SO:TSSOP-14-1EP_4.4x5mm_P0.65mm" (at 209.55 102.87 0)
+    (property "Footprint" "Package_SO:TSSOP-16_4.4x5mm_P0.65mm" (at 209.55 102.87 0)
       (effects (font (size 1.27 1.27)) (justify bottom) hide)
     )
@@
         (path "/0c53b8cf-b94b-444b-8930-5f445eddf0f0/2f1a03b0-7946-4e7c-ad47-38a79c8ba450"
           (reference "R20") (unit 1)
+        )
+      )
+    )
+  )
+  (symbol (lib_id "power:GNDD") (at 175.26 102.87 0) (unit 1)
+    (in_bom yes) (on_board yes) (dnp no) (fields_autoplaced)
+    (property "Reference" "#PWR012" (at 175.26 109.22 0)
+      (effects (font (size 1.27 1.27)) hide)
+    )
+    (property "Value" "GNDD" (at 175.26 106.68 0)
+      (effects (font (size 1.27 1.27)))
+    )
+    (property "Footprint" "" (at 175.26 102.87 0)
+      (effects (font (size 1.27 1.27)) hide)
+    )
+    (property "Datasheet" "" (at 175.26 102.87 0)
+      (effects (font (size 1.27 1.27)) hide)
+    )
+    (pin "1")
+    (instances
+      (project "LC_meter"
+        (path "/0c53b8cf-b94b-444b-8930-5f445eddf0f0"
+          (reference "#PWR012") (unit 1)
+        )
+        (path "/0c53b8cf-b94b-444b-8930-5f445eddf0f0/2f1a03b0-7946-4e7c-ad47-38a79c8ba450"
+          (reference "#PWR024") (unit 1)
         )
       )
@@
         )
       )
-    )
-  )
-  (symbol (lib_id "power:GNDA") (at 175.26 102.87 0) (unit 1)
-    (in_bom yes) (on_board yes) (dnp no) (fields_autoplaced)
-    (property "Reference" "#PWR024" (at 175.26 109.22 0)
-      (effects (font (size 1.27 1.27)) hide)
-    )
-    (property "Value" "GNDA" (at 175.26 107.95 0)
-      (effects (font (size 1.27 1.27)))
-    )
-    (property "Footprint" "" (at 175.26 102.87 0)
-      (effects (font (size 1.27 1.27)) hide)
-    )
-    (property "Datasheet" "" (at 175.26 102.87 0)
-      (effects (font (size 1.27 1.27)) hide)
-    )
-    (pin "1")
-    (instances
-      (project "LC_meter"
-        (path "/0c53b8cf-b94b-444b-8930-5f445eddf0f0/2f1a03b0-7946-4e7c-ad47-38a79c8ba450"
-          (reference "#PWR024") (unit 1)
-        )
-      )

Commit message: stability
Parts:
- R?: value 330+/-0.1% -> 2.5k+/-0.1%
- R?: value 1e3+/-0.1% -> 250+/-0.1%
Changed lines of the file:
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@@
       (effects (font (size 1.27 1.27)) (justify left))
     )
-    (property "Value" "330+/-0.1%" (at 127 168.91 90)
+    (property "Value" "2.5k+/-0.1%" (at 127 168.91 90)
       (effects (font (size 1.27 1.27)) (justify left))
     )
@@
       (effects (font (size 1.27 1.27)) (justify left))
     )
-    (property "Value" "1e3+/-0.1%" (at 127 158.75 90)
-      (effects (font (size 1.27 1.27)) (justify left))
-    )
+    (property "Value" "250+/-0.1%" (at 127 158.75 90)
+      (effects (font (size 1.27 1.27)) (justify left))
+    )

Commit message: more layout
Parts:
- C13, C14, R? (x2): value TBD -> PNU
- C6, C7: value C -> PNU
Changed lines of the file:
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@@
       (effects (font (size 1.27 1.27)))
     )
-    (property "Value" "C" (at 114.3 151.13 90)
+    (property "Value" "PNU" (at 114.3 151.13 90)
       (effects (font (size 1.27 1.27)))
     )
@@
       (effects (font (size 1.27 1.27)) (justify left))
     )
-    (property "Value" "TBD" (at 118.11 189.23 90)
+    (property "Value" "PNU" (at 118.11 189.23 90)
       (effects (font (size 1.27 1.27)) (justify left))
     )
@@
       (effects (font (size 1.27 1.27)) (justify left))
     )
-    (property "Value" "TBD" (at 118.11 179.07 90)
+    (property "Value" "PNU" (at 118.11 179.07 90)
       (effects (font (size 1.27 1.27)) (justify left))
     )
@@
       (effects (font (size 1.27 1.27)))
     )
-    (property "Value" "C" (at 114.3 161.29 90)
+    (property "Value" "PNU" (at 115.57 161.29 90)
       (effects (font (size 1.27 1.27)))
     )
@@
       (effects (font (size 1.27 1.27)))
     )
-    (property "Value" "TBD" (at 115.57 181.61 90)
+    (property "Value" "PNU" (at 115.57 181.61 90)
       (effects (font (size 1.27 1.27)))
     )
@@
       (effects (font (size 1.27 1.27)))
     )
-    (property "Value" "TBD" (at 115.57 171.45 90)
-      (effects (font (size 1.27 1.27)))
-    )
+    (property "Value" "PNU" (at 115.57 171.45 90)
+      (effects (font (size 1.27 1.27)))
+    )

Commit message: general work
Parts:
- C13, C14, C6, C7, R? (x2): now not fitted
- renumbered TP1 to TP?
Changed lines of the file:
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@@
   )
   (symbol (lib_id "Device:C") (at 111.76 152.4 90) (unit 1)
-    (in_bom yes) (on_board yes) (dnp no)
+    (in_bom yes) (on_board yes) (dnp yes)
     (property "Reference" "C6" (at 109.22 151.13 90)
       (effects (font (size 1.27 1.27)))
     )
-    (property "Value" "PNU" (at 114.3 151.13 90)
+    (property "Value" "PNU" (at 115.57 151.13 90)
       (effects (font (size 1.27 1.27)))
     )
@@
   (symbol (lib_id "Connector:TestPoint_Alt") (at 158.75 119.38 90) (unit 1)
     (in_bom yes) (on_board yes) (dnp no) (fields_autoplaced)
-    (property "Reference" "TP1" (at 155.448 114.3 90)
+    (property "Reference" "TP?" (at 155.448 114.3 90)
       (effects (font (size 1.27 1.27)))
     )
@@
       (project "LC_meter"
         (path "/0c53b8cf-b94b-444b-8930-5f445eddf0f0"
-          (reference "TP1") (unit 1)
+          (reference "TP?") (unit 1)
         )
         (path "/0c53b8cf-b94b-444b-8930-5f445eddf0f0/2f1a03b0-7946-4e7c-ad47-38a79c8ba450"
@@
   (symbol (lib_id "Connector:TestPoint_Alt") (at 118.11 119.38 0) (unit 1)
     (in_bom yes) (on_board yes) (dnp no) (fields_autoplaced)
-    (property "Reference" "TP1" (at 120.65 114.808 0)
+    (property "Reference" "TP?" (at 120.65 114.808 0)
       (effects (font (size 1.27 1.27)) (justify left))
     )
@@
       (project "LC_meter"
         (path "/0c53b8cf-b94b-444b-8930-5f445eddf0f0"
-          (reference "TP1") (unit 1)
+          (reference "TP?") (unit 1)
         )
         (path "/0c53b8cf-b94b-444b-8930-5f445eddf0f0/2f1a03b0-7946-4e7c-ad47-38a79c8ba450"
@@
   (symbol (lib_id "Connector:TestPoint_Alt") (at 97.79 36.83 0) (unit 1)
     (in_bom yes) (on_board yes) (dnp no) (fields_autoplaced)
-    (property "Reference" "TP1" (at 100.33 32.258 0)
+    (property "Reference" "TP?" (at 100.33 32.258 0)
       (effects (font (size 1.27 1.27)) (justify left))
     )
@@
       (project "LC_meter"
         (path "/0c53b8cf-b94b-444b-8930-5f445eddf0f0"
-          (reference "TP1") (unit 1)
+          (reference "TP?") (unit 1)
         )
         (path "/0c53b8cf-b94b-444b-8930-5f445eddf0f0/2f1a03b0-7946-4e7c-ad47-38a79c8ba450"
@@
   )
   (symbol (lib_id "Device:R_US") (at 111.76 187.96 90) (unit 1)
-    (in_bom yes) (on_board yes) (dnp no)
+    (in_bom yes) (on_board yes) (dnp yes)
     (property "Reference" "R?" (at 109.22 189.23 90)
       (effects (font (size 1.27 1.27)) (justify left))
@@
   (symbol (lib_id "power:GNDD") (at 175.26 102.87 0) (unit 1)
     (in_bom yes) (on_board yes) (dnp no) (fields_autoplaced)
-    (property "Reference" "#PWR012" (at 175.26 109.22 0)
+    (property "Reference" "#PWR?" (at 175.26 109.22 0)
       (effects (font (size 1.27 1.27)) hide)
     )
@@
       (project "LC_meter"
         (path "/0c53b8cf-b94b-444b-8930-5f445eddf0f0"
-          (reference "#PWR012") (unit 1)
+          (reference "#PWR?") (unit 1)
         )
         (path "/0c53b8cf-b94b-444b-8930-5f445eddf0f0/2f1a03b0-7946-4e7c-ad47-38a79c8ba450"
@@
   )
   (symbol (lib_id "Device:R_US") (at 111.76 177.8 90) (unit 1)
-    (in_bom yes) (on_board yes) (dnp no)
+    (in_bom yes) (on_board yes) (dnp yes)
     (property "Reference" "R?" (at 109.22 179.07 90)
       (effects (font (size 1.27 1.27)) (justify left))
@@
   )
   (symbol (lib_id "Device:C") (at 111.76 162.56 90) (unit 1)
-    (in_bom yes) (on_board yes) (dnp no)
+    (in_bom yes) (on_board yes) (dnp yes)
     (property "Reference" "C7" (at 109.22 161.29 90)
       (effects (font (size 1.27 1.27)))
@@
   (symbol (lib_id "Connector:TestPoint_Alt") (at 107.95 143.51 0) (unit 1)
     (in_bom yes) (on_board yes) (dnp no) (fields_autoplaced)
-    (property "Reference" "TP1" (at 110.49 138.938 0)
+    (property "Reference" "TP?" (at 110.49 138.938 0)
       (effects (font (size 1.27 1.27)) (justify left))
     )
@@
       (project "LC_meter"
         (path "/0c53b8cf-b94b-444b-8930-5f445eddf0f0"
-          (reference "TP1") (unit 1)
+          (reference "TP?") (unit 1)
         )
         (path "/0c53b8cf-b94b-444b-8930-5f445eddf0f0/2f1a03b0-7946-4e7c-ad47-38a79c8ba450"
@@
   )
   (symbol (lib_id "Device:C") (at 111.76 182.88 90) (unit 1)
-    (in_bom yes) (on_board yes) (dnp no)
+    (in_bom yes) (on_board yes) (dnp yes)
     (property "Reference" "C14" (at 107.95 181.61 90)
       (effects (font (size 1.27 1.27)))
@@
   )
   (symbol (lib_id "Device:C") (at 111.76 172.72 90) (unit 1)
-    (in_bom yes) (on_board yes) (dnp no)
+    (in_bom yes) (on_board yes) (dnp yes)
     (property "Reference" "C13" (at 107.95 171.45 90)
       (effects (font (size 1.27 1.27)))

Commit message: layout draft
Parts:
- added C?: 0.1uF, Capacitor_SMD:C_0805_2012Metric, symbol Device:C
- added R26: 2.21k, Resistor_SMD:R_0805_2012Metric, symbol Device:R_US
- added R27, R30, R31: 10k, Resistor_SMD:R_0805_2012Metric, symbol Device:R_US
- added U6: LM6142xIx, Package_DIP:DIP-8_W7.62mm, symbol Amplifier_Operational:LM6142xIx
- R15: value 10k -> 2.21k
Connections:
- net +5V: now also C?.1, R30.1, U6.8 (V+); no longer R15.1
- net GNDA: now also C?.2, R27.2, R31.1, U6.4 (V-)
- net at C13.2, C14.2, C6.2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: now also R15.2; no longer U4.2 (+IN1)
- net at R16.1, U1.12 (+): now also R15.1; no longer R15.2
- net at TP?.1, U1.6 (-), U1.7: now also R26.2; no longer U4.3 (+IN0)
- net at U1.13 (-), U1.14: now also U4.2 (+IN1)
- new net: R30.2, R31.2, U6.5 (+)
- new net: U6.6 (-), U6.7
- new net: U4.3 (+IN0), U6.1, U6.2 (-)
- new net: R26.1, R27.1, U6.3 (+)
Other:
- title: Inductance and Capacitance Meter Analog Front End -> LCR Meter Analog Front End
- moved on the sheet: C1, C11, C13, C14, C6, C7, C8, C9, C?, J1, J2, J4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

Commit message: more work on algorithm
Parts:
- C1, C11, C8, C? (x2): Distributor (none) -> DIGIKEY; Distributor Part # (none) -> 1276-1003-1-ND; Part # (none) -> CL21B104KBCNNNC; Unit Price (none) -> 0.1
- C13, C14, C6, C7, R? (x2): Distributor (none) -> N/A; Distributor Part # (none) -> N/A; Part # (none) -> N/A; Price (none) -> N/A; Unit Price (none) -> N/A
- C9: Distributor (none) -> DIGIKEY; Distributor Part # (none) -> 1276-1096-1-ND; Part # (none) -> CL21A106KOQNNNE; Unit Price (none) -> 0.1
- C? (x3): Distributor (none) -> DIGIKEY; Distributor Part # (none) -> 1276-1261-1-ND; Part # (none) -> CL21C101JCANNNC; Unit Price (none) -> 0.1
- R1, R16, R2, R27: value 10k -> 10k+/-0.1%; Distributor (none) -> DIGIKEY; Distributor Part # (none) -> P10KDACT-ND; Part # (none) -> ERA-6AEB103V; Unit Price (none) -> 0.32
- R15, R26: value 2.21k -> 2.21k+/-0.1%; Distributor (none) -> DIGIKEY; Distributor Part # (none) -> P2.21KDACT-ND; Part # (none) -> ERA-6AEB2211V; Unit Price (none) -> 0.32
- R17, R30, R31: Distributor (none) -> DIGIKEY; Distributor Part # (none) -> RMCF0805FT10K0CT-ND; Part # (none) -> RMCF0805FT10K0; Unit Price (none) -> 0.1
- R18: Distributor (none) -> DIGIKEY; Distributor Part # (none) -> RMCF0805FT1K00CT-ND; Part # (none) -> RMCF0805FT1K00; Unit Price (none) -> 0.1
- R?: Distributor (none) -> DIGIKEY; Distributor Part # (none) -> 738-RMCF0805FT187KCT-ND; Part # (none) -> RMCF0805FT187K; Unit Price (none) -> 0.1
- R? (x4): Distributor (none) -> DIGIKEY; Distributor Part # (none) -> RMCF0805FT13K0CT-ND; Part # (none) -> RMCF0805FT13K0; Unit Price (none) -> 0.1
- R?: value 50k+/-0.1% -> 49.9k+/-0.1%; Distributor (none) -> DIGIKEY; Distributor Part # (none) -> P49.9KDACT-ND; Part # (none) -> ERA-6AEB4992V; Unit Price (none) -> 0.32
- R?: value 2.5k+/-0.1% -> 2.49k+/-0.1%; Distributor (none) -> DIGIKEY; Distributor Part # (none) -> 13-RP0805BRD072K49LCT-ND; Part # (none) -> RP0805BRD072K49L; Unit Price (none) -> 0.48
- R?: value 500k+/-0.1% -> 499k+/-0.1%; Distributor (none) -> DIGIKEY; Distributor Part # (none) -> RG20P499KBCT-ND; Part # (none) -> RG2012P-4993-B-T5; Unit Price (none) -> 0.48
- R?: value 5k+/-0.1% -> 4.99k+/-0.1%; Distributor (none) -> DIGIKEY; Distributor Part # (none) -> P4.99KDACT-ND; Part # (none) -> ERA-6AEB4991V; Unit Price (none) -> 0.32
- R?: value 500+/-0.1% -> 499+/-0.1%; Distributor (none) -> DIGIKEY; Distributor Part # (none) -> RG20P499BCT-ND; Part # (none) -> RG2012P-4990-B-T5; Unit Price (none) -> 0.48
- R?: value 250+/-0.1% -> 249+/-0.1%; Distributor (none) -> DIGIKEY; Distributor Part # (none) -> P20523CT-ND; Part # (none) -> ERJ-PB6B2490V; Unit Price (none) -> 0.37
- R?: Distributor (none) -> DIGIKEY; Distributor Part # (none) -> RMCF0805FT6K49CT-ND; Part # (none) -> RMCF0805FT6K49; Unit Price (none) -> 0.1
- TP? (x4): Distributor (none) -> DIGIKEY; Distributor Part # (none) -> 36-4952-ND; Part # (none) -> 4952; Unit Price (none) -> 0.26
- U4: Availability In Stock -> (none); Check_prices https://www.snapeda.com/parts/ADS8328IPW/Texas+Instruments/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 -> (none); MF Texas Instruments -> (none); MP ADS8328IPW -> (none); Package TSSOP-16 Texas Instruments -> (none); Price None -> (none); Purchase-URL https://www.snapeda.com/api/url_track_click_mouser/?unipart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 -> (none); SnapEDA_Link https://www.snapeda.com/parts/ADS8328IPW/Texas+Instruments/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 -> (none)
Other:
- moved on the sheet: C1, C?, R15, R16, R26, R?, TP?, U1A, U1E

Commit message: finished algorithm
Connections:
- net CONVST: now reaches U4.9 (CONVST)
- no-connect marks 1 -> 0
Changed lines of the file:
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@@
   (junction (at 55.88 26.67) (diameter 0) (color 0 0 0 0)
   )
-  (no_connect (at 209.55 114.3))
   (wire (pts (xy 81.28 172.72) (xy 82.55 172.72))
     (stroke (width 0) (type default))
@@
   )
   (wire (pts (xy 191.77 104.14) (xy 193.04 104.14))
+    (stroke (width 0) (type default))
+  )
+  (wire (pts (xy 208.28 114.3) (xy 209.55 114.3))
     (stroke (width 0) (type default))
   )
@@
     (effects (font (size 1.27 1.27)) (justify right))
   )
+  (hierarchical_label "CONVST" (shape input) (at 208.28 114.3 180) (fields_autoplaced)
+    (effects (font (size 1.27 1.27)) (justify right))
+  )

Commit message: boms
Parts:
- J1: Distributor (none) -> DIGIKEY; Distributor Part # (none) -> ED10561-ND; Part # (none) -> OSTVN02A150; Unit Price (none) -> 1.08
- J2, J4, J6, J7: Distributor (none) -> DIGIKEY; Distributor Part # (none) -> ED10563-ND; Part # (none) -> OSTVN04A150; Unit Price (none) -> 1.64
- U1: Distributor (none) -> DIGIKEY; Distributor Part # (none) -> LM6144BIN/NOPB-ND; Part # (none) -> LM6144BIN/NOPB; Unit Price (none) -> 9.01
- U2: Distributor (none) -> DIGIKEY; Distributor Part # (none) -> 296-41427-1-ND; Part # (none) -> LM4030CMF-4.096/NOPB; Unit Price (none) -> 1.7
- U4: Distributor (none) -> DIGIKEY; Distributor Part # (none) -> 296-19766-ND; Part # (none) -> ADS8328IPW; Unit Price (none) -> 14.78
- U6: Distributor (none) -> MOUSER; Distributor Part # (none) -> 926-LM6142BIN/NOPB; Part # (none) -> LM6142BIN/NOPB; Unit Price (none) -> 5.58
