File: peak_detector/ecad/peak_detector.kicad_sch (KiCad schematic)
At the start: 24 parts, among them J1 Input 1, J2 Input 2, J3 Discharge 1, J4 Discharge 2, Q1 2N7002, Q2 2N7002, U1 MCP6024

Commit message: varius work
Parts:
- removed Q1, Q2: 2N7002, Package_TO_SOT_SMD:SOT-23, symbol Transistor_FET:2N7002
- added D5: 1N5817, Diode_THT:D_DO-41_SOD81_P10.16mm_Horizontal, symbol Diode:1N5817
- added H1, H2, H3, H4: M3, MountingHole:MountingHole_3.2mm_M3_Pad_Via, symbol Mechanical:MountingHole_Pad
- added J5: Out 1, TerminalBlock_Phoenix:TerminalBlock_Phoenix_MPT-0,5-2-2.54_1x02_P2.54mm_Horizontal, symbol Connector:Screw_Terminal_01x02
- added J6: Out 2, TerminalBlock_Phoenix:TerminalBlock_Phoenix_MPT-0,5-2-2.54_1x02_P2.54mm_Horizontal, symbol Connector:Screw_Terminal_01x02
- added J7: Power, TerminalBlock_Phoenix:TerminalBlock_Phoenix_MPT-0,5-2-2.54_1x02_P2.54mm_Horizontal, symbol Connector:Screw_Terminal_01x02
- added Q1, Q2: 2N7000, Package_TO_SOT_THT:TO-92_Inline, symbol Transistor_FET:2N7000
- added R11, R12, R13, R14: 1k, Resistor_THT:R_Axial_DIN0207_L6.3mm_D2.5mm_P7.62mm_Horizontal, symbol Device:R_US
- added R15, R16: 100, symbol Device:R_US
- C1: footprint (none) -> Capacitor_THT:C_Disc_D6.0mm_W2.5mm_P5.00mm; Digikey Part # (none) -> BC2665CT-ND; Part # (none) -> K104K10X7RF5UH5; Unit Price (none) -> 0.25
- C2, C3: footprint (none) -> Capacitor_THT:C_Disc_D6.0mm_W2.5mm_P5.00mm
- D1, D2, D3, D4: footprint (none) -> Diode_SMD:D_SOD-323; Digikey Part # (none) -> 1514-CMDD6001TRPBFREECT-ND; Part # (none) -> CMDD6001; Unit Price (none) -> 0.68
- J1, J2, J3, J4: footprint (none) -> TerminalBlock_Phoenix:TerminalBlock_Phoenix_MPT-0,5-2-2.54_1x02_P2.54mm_Horizontal
- R1, R2: footprint (none) -> Resistor_THT:R_Axial_DIN0207_L6.3mm_D2.5mm_P7.62mm_Horizontal; Digikey Part # (none) -> 13-MFR-25FRF52-100RCT-ND; Part # (none) -> MFR-25FRF52-100R; Unit Price (none) -> 0.1
- R10, R9: footprint (none) -> Resistor_THT:R_Axial_DIN0207_L6.3mm_D2.5mm_P7.62mm_Horizontal; Digikey Part # (none) -> CF14JT1K00CT-ND; Part # (none) -> CF14JT1K00; Unit Price (none) -> 0.1
- R3, R4: value R_US -> 1k; footprint (none) -> Resistor_THT:R_Axial_DIN0207_L6.3mm_D2.5mm_P7.62mm_Horizontal; Digikey Part # (none) -> CF14JT1K00CT-ND; Part # (none) -> CF14JT1K00; Unit Price (none) -> 0.1
- R5, R6: footprint (none) -> Resistor_THT:R_Axial_DIN0207_L6.3mm_D2.5mm_P7.62mm_Horizontal; Digikey Part # (none) -> CF14JT100KCT-ND; Part # (none) -> CF14JT100K; Unit Price (none) -> 0.1
- R7, R8: footprint (none) -> Resistor_THT:R_Axial_DIN0207_L6.3mm_D2.5mm_P7.62mm_Horizontal; Digikey Part # (none) -> CF14JT10K0CT-ND; Part # (none) -> CF14JT10K0; Unit Price (none) -> 0.1
- U1: footprint (none) -> Package_DIP:DIP-14_W7.62mm; Digikey Part # (none) -> MCP6024-I/P-ND; Part # (none) -> MCP6024-I/P; Unit Price (none) -> 2.72
Connections:
- net +5V: now also D5.1 (K)
- net GND: now also H1.1, H2.1, H3.1, H4.1, J5.1 (Pin_1), J6.1 (Pin_1), J7.1 (Pin_1), Q1.1 (S), Q2.1 (S), R12.1, R14.1
- net at C2.1, R1.2, U1.10 (+): now also R15.1
- net at R3.2, U1.8, U1.9 (-): now also R11.1
- net at R10.2, R8.1: now also Q2.2 (G)
- net at R7.1, R9.2: now also Q1.2 (G)
- net at C3.1, R2.2, U1.5 (+): now also R16.1
- net at R4.2, U1.6 (-), U1.7: now also R13.1
- new net: Q2.3 (D), R16.2
- new net: J5.2 (Pin_2), R11.2, R12.2
- new net: D5.2 (A), J7.2 (Pin_2)
- new net: J6.2 (Pin_2), R13.2, R14.2
- new net: Q1.3 (D), R15.2
Other:
- moved on the sheet: C1, C2, C3, D1, D2, D3, D4, J1, J2, J3, J4, R1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
