File: electronics/rev2/ecad/LCR_meter.kicad_sch (KiCad schematic)
At the start: 46 parts, among them J1 DUT, J2 DUT, J3 SWITCH, J4 SWITCH, U1 OP179GRT, U4 ADG1408YRUZ, U5 SC0915, U6 AD8226ARZ, U7 LM4040DBZ-3, U8 OP279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

Commit message: schematic rev2 might be done
Parts:
- removed C5, C6: 0.1uF, symbol Device:C
- removed R11: 100k, symbol Device:R_US
- removed R4: 10k, symbol Device:R_US
- removed U4: ADG1408YRUZ, Package_SO:TSSOP-16_4.4x5mm_P0.65mm, symbol Analog_Switch:ADG1408YRUZ
- removed U6, U9: AD8226ARZ, AD8226ARZ:SOIC127P600X175-8N, symbol AD8226ARZ:AD8226ARZ
- removed U8: OP279, symbol Amplifier_Operational:OP279
- added C8: 0.1uF, Capacitor_SMD:C_0603_1608Metric_Pad1.08x0.95mm_HandSolder, symbol Device:C
- added U2: MCP6001R, Package_TO_SOT_SMD:SOT-23-5, symbol Amplifier_Operational:MCP6001R
- added U4: 74HC4051, Package_SO:SOIC-16_3.9x9.9mm_P1.27mm, symbol 74xx:74HC4051
- C1, C2, C3, C4, C7: footprint (none) -> Capacitor_SMD:C_0603_1608Metric_Pad1.08x0.95mm_HandSolder
- J1, J2, J3: footprint (none) -> Connector_PinHeader_2.54mm:PinHeader_1x02_P2.54mm_Vertical
- J4: footprint (none) -> Connector_PinHeader_2.54mm:PinHeader_1x03_P2.54mm_Vertical
- R1, R10, R12, R13, R14, R15, R16, R17, R18, R19, R20, R21, R22, R23, R24, R6, R7, R8, R9: footprint (none) -> Resistor_SMD:R_0603_1608Metric_Pad0.98x0.95mm_HandSolder
- R2: value 100k -> 10k; footprint (none) -> Resistor_SMD:R_0603_1608Metric_Pad0.98x0.95mm_HandSolder
- R3: value R_US -> 10k; footprint (none) -> Resistor_SMD:R_0603_1608Metric_Pad0.98x0.95mm_HandSolder
- R5: value 187k -> 249k; footprint (none) -> Resistor_SMD:R_0603_1608Metric_Pad0.98x0.95mm_HandSolder
- TP1, TP2, TP3, TP4: footprint (none) -> TestPoint:TestPoint_Pad_D1.5mm
- U5: footprint SC0915:MODULE_SC0915 -> LCR_meter_parts:MODULE_SC0915
Connections:
- net +5V: now also R2.1, C8.2, U2.2 (V+), U4.16 (VCC)
- net GND: now also R12.2, C8.1, U2.5 (V-), U4.6 (~{E}), U4.7 (VEE), U4.8 (GND); no longer R12.1
- net bit0: now also U4.11 (S0)
- net bit1: now also U4.10 (S1)
- net bit2: now also U4.9 (S2)
- net DiffAmp1/IN+: now reaches C4.2, R5.2, TP3.1
- net DiffAmp1/IN+: now also U2.1, U4.3 (A)
- net at R3.2, U5.35 (ADC_VREF), U7.1 (K): now also R2.2
- net at R10.1, TP2.1, U5.32 (GP27): now also R12.1; no longer R12.2
- net at R5.1, R6.1: now also U2.4 (-)
- net DiffAmp2/IN-: now reaches J2.1 (Pin_1), J2.2 (Pin_2), R1.2, R7.2, TP4.1, U1.1, U1.4 (-)
- net DiffAmp2/IN-: now also U2.3 (+)
- net at R16.1: now also U4.12 (A3)
- net DiffAmp1/IN-: now reaches J1.1 (Pin_1), J1.2 (Pin_2), R13.2, R14.2, R15.2, R16.2, R17.2, R18.2, R19.2
- net at R13.1: now also U4.2 (A6)
- net at R14.1: now also U4.5 (A5)
- net at R15.1: now also U4.1 (A4)
- net at R19.1: now also U4.13 (A0)
- net at R18.1: now also U4.14 (A1)
- net at R17.1: now also U4.15 (A2)
- net DiffAmp2/OUT: now reaches R10.2
- net DiffAmp1/OUT: now reaches R8.1
Other:
- added sheet DiffAmp1 (diff_amp.kicad_sch)
- added sheet DiffAmp2 (diff_amp.kicad_sch)
- moved on the sheet: C2, C3, C4, C7, J1, J2, J3, J4, R1, R10, R20, R21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

Commit message: rev2 design work
Parts:
- removed C7: 0.1uF, Capacitor_SMD:C_0603_1608Metric_Pad1.08x0.95mm_HandSolder, symbol Device:C
- removed R19: 49.9, Resistor_SMD:R_0603_1608Metric_Pad0.98x0.95mm_HandSolder, symbol Device:R_US
- removed U1: OP179GRT, Package_TO_SOT_SMD:SOT-23-5, symbol Amplifier_Operational:OP179GRT
- removed U2: MCP6001R, Package_TO_SOT_SMD:SOT-23-5, symbol Amplifier_Operational:MCP6001R
- added H1, H2, H3, H4: M3, MountingHole:MountingHole_3.2mm_M3_Pad_Via, symbol Mechanical:MountingHole_Pad
- added U1: MCP6002-xSN, Package_SO:SOIC-8_3.9x4.9mm_P1.27mm, symbol Amplifier_Operational:MCP6002-xSN
- C1, C8: Digikey Part # (none) -> 311-1088-1-ND; Part # (none) -> CC0603KRX7R7BB104; Unit Price 100x (none) -> 0.02; Unit Price 1x (none) -> 0.1
- C2, C3, C4: Digikey Part # (none) -> 1276-1008-1-ND; Part # (none) -> CL10C101JB8NNNC; Unit Price 100x (none) -> 0.0116; Unit Price 1x (none) -> 0.1
- J1, J2, J3: Digikey Part # (none) -> 732-5315-ND; Part # (none) -> 61300211121; Unit Price 100x (none) -> 0.071; Unit Price 1x (none) -> 0.13
- J4: value SWITCH -> INPUT SWITCH; Digikey Part # (none) -> 732-5316-ND; Part # (none) -> 61300311121; Unit Price 100x (none) -> 0.071; Unit Price 1x (none) -> 0.13
- R1, R6, R7: value 6.49k -> 6.49k+/-0.1%; Digikey Part # (none) -> P6.49KHCT-ND; Part # (none) -> ERJ-3EKF6491V; Unit Price 100x (none) -> 0.0163; Unit Price 1x (none) -> 0.1
- R10, R8: value 6.81k -> 6.81k+/-0.1%; Digikey Part # (none) -> 311-6.81KHRCT-ND; Part # (none) -> RC0603FR-076K81L; Unit Price 100x (none) -> 0.00650; Unit Price 1x (none) -> 0.1
- R12, R20, R21, R9: value 10k -> 10k+/-0.1%; Digikey Part # (none) -> YAG1236CT-ND; Part # (none) -> RT0603BRD0710KL; Unit Price 100x (none) -> 0.073; Unit Price 1x (none) -> 0.14
- R13: value 49.9M -> 49.9M+/-0.1%; now not fitted; now left out of the parts list
- R14: value 4.99M -> 4.99M+/-0.1%; Digikey Part # (none) -> RMCF0603FT4M99CT-ND; Part # (none) -> RMCF0603FT4M99; Unit Price 100x (none) -> 0.01080; Unit Price 1x (none) -> 0.1
- R15: value 499k -> 499k+/-0.1%; Digikey Part # (none) -> 2019-RN73R1JTTD4993B25CT-ND; Part # (none) -> RN73R1JTTD4993B25; Unit Price 100x (none) -> 0.1091; Unit Price 1x (none) -> 0.21
- R16: value 49.9k -> 49.9k+/-0.1%; Digikey Part # (none) -> P49.9KDBCT-ND; Part # (none) -> ERA-3AEB4992V; Unit Price 100x (none) -> 0.0697; Unit Price 1x (none) -> 0.13
- R17: value 4.99k -> 4.99k+/-0.1%; Digikey Part # (none) -> P4.99KDBCT-ND; Part # (none) -> ERA-3AEB4991V; Unit Price 100x (none) -> 0.0697; Unit Price 1x (none) -> 0.13
- R18: value 499 -> 499+/-0.1%; Digikey Part # (none) -> P499DBCT-ND; Part # (none) -> ERA-3AEB4990V; Unit Price 100x (none) -> 0.0715; Unit Price 1x (none) -> 0.14
- R2, R22, R23, R24, R3: Digikey Part # (none) -> 311-10.0KHRCT-ND; Part # (none) -> RC0603FR-0710KL; Unit Price 100x (none) -> 0.0093; Unit Price 1x (none) -> 0.1
- R5: value 249k -> 249k+/-0.1%; Digikey Part # (none) -> P249KDBCT-ND; Part # (none) -> ERA-3AEB2493V; Unit Price 100x (none) -> 0.0697; Unit Price 1x (none) -> 0.13
- U4: Digikey Part # (none) -> 296-14530-1-ND; Part # (none) -> CD74HC4051M96; Unit Price 100x (none) -> 0.4; Unit Price 1x (none) -> 0.1973
- U7: Digikey Part # (none) -> 296-38730-1-ND; Part # (none) -> LM4040AIM3X-3.0/NOPB; Unit Price 100x (none) -> 1.1303; Unit Price 1x (none) -> 2.02
Connections:
- net +5V: now also U1.8 (V+)
- net DiffAmp1/IN+: now also U1.1
- net DiffAmp1/OUT: now also R8.2, TP1.1; no longer R8.1
- net GND: now also H1.1, H2.1, H3.1, H4.1, U1.4 (V-)
- net at R20.2, R21.1: now also U1.5 (+)
- net at R9.2, U5.31 (GP26): now also R8.1; no longer R8.2, TP1.1
- net at R5.1, R6.1: now also U1.2 (-)
- net at R16.1: now also U4.15 (A2); no longer U4.12 (A3)
- net at R18.1: now also U4.13 (A0); no longer U4.14 (A1)
- net at R15.1: now also U4.12 (A3); no longer U4.1 (A4)
- net at R17.1: now also U4.14 (A1); no longer U4.15 (A2)
- net at U4.2 (A6): no longer R13.1
- net at R14.1: now also U4.1 (A4); no longer U4.5 (A5)
- net DiffAmp2/IN- renamed DiffAmp1/REF
- net DiffAmp1/REF: now also U1.3 (+), U1.6 (-), U1.7
- new net: R13.1, U4.5 (A5)
- no-connect marks 29 -> 30
Other:
- sheet DiffAmp1 ports: added REF; removed none
- sheet DiffAmp2 ports: added REF; removed none
- moved on the sheet: C2, C3, C4, C8, J1, J2, J3, J4, R1, R10, R12, R14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
