File: electronics/rev2/ecad/diff_amp.kicad_sch (KiCad schematic)
At the start: 8 parts, among them U3 LM6144xIx

Commit message: rev2 design work
Parts:
- C5: Digikey Part # (none) -> 311-1088-1-ND; Part # (none) -> CC0603KRX7R7BB104; Unit Price 100x (none) -> 0.02; Unit Price 1x (none) -> 0.1
- R25, R26, R27, R30: Digikey Part # (none) -> YAG1236CT-ND; Part # (none) -> RT0603BRD0710KL; Unit Price 100x (none) -> 0.073; Unit Price 1x (none) -> 0.14
- R28, R34: Digikey Part # (none) -> 311-10.0KHRCT-ND; Part # (none) -> RC0603FR-0710KL; Unit Price 100x (none) -> 0.0093; Unit Price 1x (none) -> 0.1
- U3: Digikey Part # (none) -> 296-35226-1-ND; Part # (none) -> LM6144BIMX/NOPB; Unit Price 100x (none) -> 5.137; Unit Price 1x (none) -> 8.34
Connections:
- net GND: no longer R25.1
- new net REF: R25.1
